File: Pcb_geral/pcb_geral/_autosave-pcb_geral.kicad_pcb (KiCad board)
At the start: 2 copper layers, 21 parts, among them U1 LM2594M-3.3, U2 LM2596S-5, U3 STM32F103C6Tx, U4 TJA1051T, Y2 8Mhz

Commit message: atualizacoes, sem grandes modificacoes
Parts:
- moved U4 58.0 mm to (101.4, 66.5)
- moved C1 32.6 mm to (132.7, 50.2)
- moved U1 32.6 mm to (124.3, 49.7)
- moved C3 32.6 mm to (125.5, 42.2)
- moved D1 32.6 mm to (132.0, 42.3)
- moved L2 30.0 mm to (87.5, 52.4), turned to 90 degrees
- moved C8 27.4 mm to (89.5, 41.6), turned to 0 degrees
- moved C7 26.1 mm to (113.3, 53.7), turned to -90 degrees
- moved D1 25.9 mm to (113.3, 43.2), turned to 0 degrees
- moved Prog1 25.3 mm to (152.5, 52.4), turned to 90 degrees
- moved C5 14.2 mm to (143.0, 52.8)
- moved U2 5.74 mm to (100.4, 51.0), turned to -90 degrees
- moved L1 4.50 mm to (143.8, 45.2)
