File: Pcb_geral/pcb_geral/_autosave-pcb_geral.kicad_sch (KiCad schematic)
At the start: 30 parts, among them U1 LM2594M-3.3, U2 LM2596S-5, U3 STM32F103C6Tx

Commit message: atualizacoes, sem grandes modificacoes
Parts:
- gave numbers to parts that had none: 17
